File: pcb/0xB2.kicad_sch (KiCad schematic)
At the start: 40 parts, among them J1 USB_C_Receptacle_USB2.0, J2 Conn_01x12, J3 Conn_01x05, J4 Conn_01x12, J5 Conn_01x02, SW1 SW_Push, SW2 SW_Push, U1 RP2040, U2 GD25Q80CEIGR, U3 XC6210B332MR-G, Y1 Crystal_GND24

Commit message: switch to M13
Parts:
- J1: footprint 0xLib_USB_Type-C:USB_C_Receptacle_HRO_TYPE-C-31-M-14 -> drawings:HRO-TYPE-C-31-M-13
Changed lines of the file:
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@@
     (property "Reference" "J1" (id 0) (at 35.56 29.21 0))
     (property "Value" "USB_C_Receptacle_USB2.0" (id 1) (at 35.56 31.75 0))
-    (property "Footprint" "0xLib_USB_Type-C:USB_C_Receptacle_HRO_TYPE-C-31-M-14" (id 2) (at 39.37 52.07 0)
+    (property "Footprint" "drawings:HRO-TYPE-C-31-M-13" (id 2) (at 39.37 52.07 0)
       (effects (font (size 1.27 1.27)) hide)
     )
@@
     )
     (path "/6125bb34-31fe-49ed-b2ab-61dab24d450a"
-      (reference "J1") (unit 1) (value "USB_C_Receptacle_USB2.0") (footprint "0xLib_USB_Type-C:USB_C_Receptacle_HRO_TYPE-C-31-M-14")
+      (reference "J1") (unit 1) (value "USB_C_Receptacle_USB2.0") (footprint "drawings:HRO-TYPE-C-31-M-13")
     )
     (path "/44683f1e-d2b9-4133-9a9d-84586c32a6a2"
